Commit message: Add initial position config file for mock hardware

File: kuka_rsi_driver/urdf/kuka_rsi_driver.ros2_control.xacro (robot description, xacro)
@@ -1,8 +1,10 @@
 <?xml version="1.0"?>
 <robot xmlns:xacro="http://www.ros.org/wiki/xacro">
-  <xacro:macro name="kuka_rsi_driver_control_joint" params="name">
+  <xacro:macro name="kuka_rsi_driver_control_joint" params="name initial_position">
     <joint name="${name}">
       <command_interface name="position" />
-      <state_interface name="position" />
+      <state_interface name="position">
+        <param name="initial_value">${initial_position}</param>
+      </state_interface>
       <state_interface name="effort" />
     </joint>
@@ -12,4 +14,5 @@
     prefix
     use_mock_hardware:=false
+    initial_positions:=${dict(joint_a1=0.0,joint_a2=0.0,joint_a3=0.0,joint_a4=0.0,joint_a5=0.0,joint_a6=0.0)}
     rsi_listen_ip
     rsi_listen_port:=49152
@@ -26,10 +29,10 @@
         </xacro:unless>
       </hardware>
-      <xacro:kuka_rsi_driver_control_joint name="${prefix}joint_a1" />
-      <xacro:kuka_rsi_driver_control_joint name="${prefix}joint_a2" />
-      <xacro:kuka_rsi_driver_control_joint name="${prefix}joint_a3" />
-      <xacro:kuka_rsi_driver_control_joint name="${prefix}joint_a4" />
-      <xacro:kuka_rsi_driver_control_joint name="${prefix}joint_a5" />
-      <xacro:kuka_rsi_driver_control_joint name="${prefix}joint_a6" />
+      <xacro:kuka_rsi_driver_control_joint name="${prefix}joint_a1" initial_position="${initial_positions['joint_a1']}" />
+      <xacro:kuka_rsi_driver_control_joint name="${prefix}joint_a2" initial_position="${initial_positions['joint_a2']}" />
+      <xacro:kuka_rsi_driver_control_joint name="${prefix}joint_a3" initial_position="${initial_positions['joint_a3']}" />
+      <xacro:kuka_rsi_driver_control_joint name="${prefix}joint_a4" initial_position="${initial_positions['joint_a4']}" />
+      <xacro:kuka_rsi_driver_control_joint name="${prefix}joint_a5" initial_position="${initial_positions['joint_a5']}" />
+      <xacro:kuka_rsi_driver_control_joint name="${prefix}joint_a6" initial_position="${initial_positions['joint_a6']}" />
       <sensor name="${prefix}tcp">
         <state_interface name="position.x">

File: kuka_rsi_driver/urdf/test_description.urdf.xacro (robot description, xacro)
@@ -6,7 +6,10 @@
   <xacro:arg name="macro_name" default="" />
   <xacro:arg name="use_mock_hardware" default="false" />
+  <xacro:arg name="initial_positions_file" default="$(find kuka_rsi_driver)/config/initial_positions.yaml" />
   <xacro:arg name="rsi_listen_ip" default="127.0.0.1" />
   <xacro:arg name="rsi_listen_port" default="49152" />
   <xacro:arg name="prefix" default="" />
+  <!-- Convert argument to property so it can be used in a function -->
+  <xacro:property name="initial_positions_file" default="$(arg initial_positions_file)" />
   <!-- Include robot description and invoke macro -->
   <xacro:property name="description_package" value="$(arg description_package)" />
@@ -19,4 +22,5 @@
     prefix="$(arg prefix)"
     use_mock_hardware="$(arg use_mock_hardware)"
+    initial_positions="${xacro.load_yaml(initial_positions_file)}"
     rsi_listen_ip="$(arg rsi_listen_ip)"
     rsi_listen_port="$(arg rsi_listen_port)"

Commit message: Add option to use mock hardware (#12)
* Add support for mock_components

* Add initial position config file for mock hardware

* Add mock hardware to test matrix

* Remove incorrect dependency

mock_components is part of hardware_interface

File: kuka_rsi_driver/urdf/kuka_rsi_driver.ros2_control.xacro (robot description, xacro)
@@ -1,8 +1,10 @@
 <?xml version="1.0"?>
 <robot xmlns:xacro="http://www.ros.org/wiki/xacro">
-  <xacro:macro name="kuka_rsi_driver_control_joint" params="name">
+  <xacro:macro name="kuka_rsi_driver_control_joint" params="name initial_position">
     <joint name="${name}">
       <command_interface name="position" />
-      <state_interface name="position" />
+      <state_interface name="position">
+        <param name="initial_value">${initial_position}</param>
+      </state_interface>
       <state_interface name="effort" />
     </joint>
@@ -11,4 +13,6 @@
     name
     prefix
+    use_mock_hardware:=false
+    initial_positions:=${dict(joint_a1=0.0,joint_a2=0.0,joint_a3=0.0,joint_a4=0.0,joint_a5=0.0,joint_a6=0.0)}
     rsi_listen_ip
     rsi_listen_port:=49152
@@ -16,28 +20,51 @@
     <ros2_control name="${name}" type="system">
       <hardware>
-        <plugin>kuka_rsi_driver/KukaRsiHardwareInterface</plugin>
-        <param name="listen_address">${rsi_listen_ip}</param>
-        <param name="listen_port">${rsi_listen_port}</param>
+        <xacro:if value="${use_mock_hardware}">
+          <plugin>mock_components/GenericSystem</plugin>
+        </xacro:if>
+        <xacro:unless value="${use_mock_hardware}">
+          <plugin>kuka_rsi_driver/KukaRsiHardwareInterface</plugin>
+          <param name="listen_address">${rsi_listen_ip}</param>
+          <param name="listen_port">${rsi_listen_port}</param>
+        </xacro:unless>
       </hardware>
-      <xacro:kuka_rsi_driver_control_joint name="${prefix}joint_a1" />
-      <xacro:kuka_rsi_driver_control_joint name="${prefix}joint_a2" />
-      <xacro:kuka_rsi_driver_control_joint name="${prefix}joint_a3" />
-      <xacro:kuka_rsi_driver_control_joint name="${prefix}joint_a4" />
-      <xacro:kuka_rsi_driver_control_joint name="${prefix}joint_a5" />
-      <xacro:kuka_rsi_driver_control_joint name="${prefix}joint_a6" />
+      <xacro:kuka_rsi_driver_control_joint name="${prefix}joint_a1" initial_position="${initial_positions['joint_a1']}" />
+      <xacro:kuka_rsi_driver_control_joint name="${prefix}joint_a2" initial_position="${initial_positions['joint_a2']}" />
+      <xacro:kuka_rsi_driver_control_joint name="${prefix}joint_a3" initial_position="${initial_positions['joint_a3']}" />
+      <xacro:kuka_rsi_driver_control_joint name="${prefix}joint_a4" initial_position="${initial_positions['joint_a4']}" />
+      <xacro:kuka_rsi_driver_control_joint name="${prefix}joint_a5" initial_position="${initial_positions['joint_a5']}" />
+      <xacro:kuka_rsi_driver_control_joint name="${prefix}joint_a6" initial_position="${initial_positions['joint_a6']}" />
       <sensor name="${prefix}tcp">
-        <state_interface name="position.x"/>
-        <state_interface name="position.y"/>
-        <state_interface name="position.z"/>
-        <state_interface name="orientation.x"/>
-        <state_interface name="orientation.y"/>
-        <state_interface name="orientation.z"/>
-        <state_interface name="orientation.w"/>
+        <state_interface name="position.x">
+          <param name="initial_value">0</param>
+        </state_interface>
+        <state_interface name="position.y">
+          <param name="initial_value">0</param>
+        </state_interface>
+        <state_interface name="position.z">
+          <param name="initial_value">0</param>
+        </state_interface>
+        <state_interface name="orientation.x">
+          <param name="initial_value">0</param>
+        </state_interface>
+        <state_interface name="orientation.y">
+          <param name="initial_value">0</param>
+        </state_interface>
+        <state_interface name="orientation.z">
+          <param name="initial_value">0</param>
+        </state_interface>
+        <state_interface name="orientation.w">
+          <param name="initial_value">1</param>
+        </state_interface>
       </sensor>
       <gpio name="${prefix}robot_state">
-        <state_interface name="program_state" />
+        <state_interface name="program_state">
+          <param name="initial_value">3</param>
+        </state_interface>
       </gpio>
       <gpio name="${prefix}speed_scaling">
-        <state_interface name="speed_scaling_factor" />
+        <state_interface name="speed_scaling_factor">
+          <param name="initial_value">1</param>
+        </state_interface>
       </gpio>
     </ros2_control>

File: kuka_rsi_driver/urdf/test_description.urdf.xacro (robot description, xacro)
@@ -5,7 +5,11 @@
   <xacro:arg name="description_macro_file" default="" />
   <xacro:arg name="macro_name" default="" />
+  <xacro:arg name="use_mock_hardware" default="false" />
+  <xacro:arg name="initial_positions_file" default="$(find kuka_rsi_driver)/config/initial_positions.yaml" />
   <xacro:arg name="rsi_listen_ip" default="127.0.0.1" />
   <xacro:arg name="rsi_listen_port" default="49152" />
   <xacro:arg name="prefix" default="" />
+  <!-- Convert argument to property so it can be used in a function -->
+  <xacro:property name="initial_positions_file" default="$(arg initial_positions_file)" />
   <!-- Include robot description and invoke macro -->
   <xacro:property name="description_package" value="$(arg description_package)" />
@@ -17,4 +21,6 @@
     name="$(arg macro_name)"
     prefix="$(arg prefix)"
+    use_mock_hardware="$(arg use_mock_hardware)"
+    initial_positions="${xacro.load_yaml(initial_positions_file)}"
     rsi_listen_ip="$(arg rsi_listen_ip)"
     rsi_listen_port="$(arg rsi_listen_port)"

Commit message: Add urdf macro that allows specifying passthrough components

File: kuka_rsi_driver/urdf/kuka_rsi_driver.ros2_control.xacro (robot description, xacro)
@@ -20,4 +20,29 @@
     rsi_listen_ip
     rsi_listen_port:=49152
+    ">
+    <xacro:kuka_rsi_driver_control_passthrough
+      name="${name}"
+      prefix="${prefix}"
+      rw_rate="${rw_rate}"
+      use_mock_hardware="${use_mock_hardware}"
+      mock_gpio_commands="${mock_gpio_commands}"
+      mock_sensor_commands="${mock_sensor_commands}"
+      initial_positions="${initial_positions}"
+      rsi_listen_ip="${rsi_listen_ip}"
+      rsi_listen_port="${rsi_listen_port}">
+      <empty />
+    </xacro:kuka_rsi_driver_control_passthrough>
+  </xacro:macro>
+  <xacro:macro name="kuka_rsi_driver_control_passthrough" params="
+    name
+    prefix
+    rw_rate:=0
+    use_mock_hardware:=false
+    mock_gpio_commands:=false
+    mock_sensor_commands:=false
+    initial_positions:=${dict(joint_a1=0.0,joint_a2=0.0,joint_a3=0.0,joint_a4=0.0,joint_a5=0.0,joint_a6=0.0)}
+    rsi_listen_ip
+    rsi_listen_port:=49152
+    **passthrough
     ">
     <ros2_control name="${name}" type="system" rw_rate="${rw_rate}">
@@ -73,13 +98,5 @@
         </state_interface>
       </gpio>
-      <gpio name="qcs">
-        <param name="rsi_name">QCS</param>
-        <state_interface name="sensor_unlocked">
-          <param name="rsi_name">Sensor_Unlocked</param>
-        </state_interface>
-        <state_interface name="sensor_locked">
-          <param name="rsi_name">Sensor_Locked</param>
-        </state_interface>
-      </gpio>
+      <xacro:insert_block name="passthrough" />
     </ros2_control>
   </xacro:macro>
